File: DCCH/DCCH.sch (KiCad schematic (older format))
At the start: 27 parts, among them J1 Conn_01x02, J2 Conn_01x02, J3 Conn_01x05, J4 Conn_01x05, J5 Conn_01x16, U11 SN74HC595, U12 SN74HC595, U13 SN74HC595, U21 SN754410, U22 SN754410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

Commit message: Updated schematic. One shift register to one h-bridge. Also put in resistors for unused outputs.
Parts:
- removed J5: Conn_01x16, Connector_PinHeader_2.54mm:PinHeader_1x16_P2.54mm_Vertical, symbol Connector_Generic:Conn_01x16
- added C141: 0.1 uF, Capacitor_SMD:C_0805_2012Metric, symbol Device:C
- added J5: Conn_02x08_Odd_Even, Connector_PinHeader_2.54mm:PinHeader_2x08_P2.54mm_Vertical, symbol Connector_Generic:Conn_02x08_Odd_Even
- added R111, R112, R121, R122, R131, R132, R141, R142: 1k, Resistor_THT:R_Axial_DIN0204_L3.6mm_D1.6mm_P5.08mm_Horizontal, symbol Device:R_US
- added U14: SN74HC595, Package_DIP:DIP-16_W7.62mm, symbol DCCH:SN74HC595
Connections:
- net +5V: now also C141.1, U14.16 (VCC)
- net CLEAR: now also U14.10 (~SRCLR~)
- net CON-11A: now also R111.2; no longer U22.2 (1A)
- net CON-11B: now also U21.1 (1,2EN); no longer U21.7 (2A)
- net CON-11D: now also U21.7 (2A); no longer U21.1 (1,2EN)
- net CON-11E: now also U21.9 (3,4EN); no longer U21.15 (4A)
- net CON-11G: now also U21.15 (4A); no longer U21.9 (3,4EN)
- net CON-11H: now also R112.2; no longer U22.7 (2A)
- net CON-12A: now also R121.2; no longer U23.15 (4A)
- net CON-12C: now also U22.2 (1A); no longer U22.15 (4A)
- net CON-12D: now also U22.7 (2A); no longer U22.10 (3A)
- net CON-12F: now also U22.10 (3A); no longer U23.7 (2A)
- net CON-12G: now also U22.15 (4A); no longer U23.2 (1A)
- net CON-12H: now also R122.2; no longer U23.1 (1,2EN)
- net CON-13A: now also R131.2; no longer U24.9 (3,4EN)
- net CON-13B: now also U23.1 (1,2EN); no longer U23.10 (3A)
- net CON-13C: now also U23.2 (1A); no longer U23.9 (3,4EN)
- net CON-13D: now also U23.7 (2A); no longer U24.7 (2A)
- net CON-13E: now also U23.9 (3,4EN); no longer U24.2 (1A)
- net CON-13F: now also U23.10 (3A); no longer U24.1 (1,2EN)
- net CON-13G: now also U23.15 (4A); no longer U24.15 (4A)
- net CON-13H: now also R132.2; no longer U24.10 (3A)
- net GND: now also C141.2, R111.1, R112.1, R121.1, R122.1, R131.1, R132.1, R141.1, R142.1, U14.13 (~OE~), U14.8 (GND)
- net OUT-1A: now also J5.1 (Pin_1)
- net OUT-1B: now also J5.2 (Pin_2)
- net OUT-2A: now also J5.3 (Pin_3)
- net OUT-2B: now also J5.4 (Pin_4)
- net OUT-3A: now also J5.5 (Pin_5)
- net OUT-3B: now also J5.6 (Pin_6)
- net OUT-4A: now also J5.7 (Pin_7)
- net OUT-4B: now also J5.8 (Pin_8)
- net OUT-5A: now also J5.9 (Pin_9)
- net OUT-5B: now also J5.10 (Pin_10)
- net OUT-6A: now also J5.11 (Pin_11)
- net OUT-6B: now also J5.12 (Pin_12)
- net OUT-7A: now also J5.13 (Pin_13)
- net OUT-7B: now also J5.14 (Pin_14)
- net OUT-8A: now also J5.15 (Pin_15)
- net OUT-8B: now also J5.16 (Pin_16)
- net SER-13: now also U14.14 (SER); no longer J4.1 (Pin_1)
- net SYNC: now also U14.11 (SRCLK)
- net WRITE: now also U14.12 (RCLK)
- new net CON-14A: R141.2, U14.15 (QA)
- new net CON-14B: U14.1 (QB), U24.1 (1,2EN)
- new net CON-14C: U14.2 (QC), U24.2 (1A)
- new net CON-14D: U14.3 (QD), U24.7 (2A)
- new net CON-14E: U14.4 (QE), U24.9 (3,4EN)
- new net CON-14F: U14.5 (QF), U24.10 (3A)
- new net CON-14G: U14.6 (QG), U24.15 (4A)
- new net CON-14H: R142.2, U14.7 (QH)
- new net SER-14: J4.1 (Pin_1), U14.9 (QH')
Other:
- moved on the sheet: C211, C221, C231, C241, U21, U22, U23, U24
